Commit message: Render SO101 in Viser from The Robot Studio's SO-ARM100 meshes
SO101 already opened a browser view on every command but always drew a
skeleton: no mesh source existed, and the preflight hint pointed at a
--fetch-meshes call that refused the model.

- meshes.py: SO101 mesh source pinned to SO-ARM100 eecbe3e (Apache 2.0);
  all twelve mesh names the URDF references are published there unchanged.
  `karma-viz --fetch-meshes --model SO101` now works, with provenance.
- SO101.urdf: mesh paths are package://assets/NAME like Yam.urdf, so the
  viewer resolves them from the mesh cache instead of beside the URDF.
  Kinematics and inertias unchanged.
- The mesh cache lives in meshes/ next to logs/ (git-ignored now); the
  docstring, --help and docs said ~/openpi-data/meshes, which was stale.
- The "meshes not cached" warning names the real script, karma-viz.
- docs/viser.md covers both models and `--rig so101`; README and the SO101
  guide point at the one-time fetch.
- tests: SO101 mesh names all resolve to the pinned source; the no-source
  test removes SO101's entry instead of relying on its absence.

Co-Authored-By: Claude Opus 5 <noreply@anthropic.com>

File: src/openpi_control/models/arms/SO101/SO101.urdf (robot description, URDF)
Before this commit: robot so101_new_calib, 7 links, 6 joints
Links:
- link base_link: geometry collision mesh filename=package://assets/base_motor_holder_so101_v1.stl; collision mesh filename=package://assets/base_so101_v2.stl
- link gripper_link: geometry collision mesh filename=package://assets/sts3215_03a_v1.stl; collision mesh filename=package://assets/wrist_roll_follower_so101_v1.stl
- link lower_arm_link: geometry collision mesh filename=package://assets/motor_holder_so101_wrist_v1.stl; collision mesh filename=package://assets/sts3215_03a_v1.stl
- link shoulder_link: geometry collision mesh filename=package://assets/motor_holder_so101_base_v1.stl; collision mesh filename=package://assets/rotation_pitch_so101_v1.stl
- link upper_arm_link: geometry collision mesh filename=package://assets/sts3215_03a_v1.stl; collision mesh filename=package://assets/upper_arm_so101_v1.stl
- link wrist_link: geometry collision mesh filename=package://assets/sts3215_03a_no_horn_v1.stl; collision mesh filename=package://assets/wrist_roll_pitch_so101_v2.stl
